File: AM Radio/AM Radio.kicad_pcb (KiCad board)
At the start: 4 copper layers, 100 x 100 mm, 92 parts, among them J101 CAL_O, J102 CAL_S, J103 CAL_L, J104 Antenna Input, J701 Conn_WallPlug_Earth, Q1 2N2222, Q2 2N2222, Q3 2N2222, Q301 2N2222, Q302 2N2222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

Commit message: more pcb work
Parts:
- moved T401 301.0 mm to (125.2, 102.2), turned to 90 degrees
- moved T402 279.0 mm to (125.2, 71.8), turned to 270 degrees
- moved C502 274.6 mm to (114.4, 81.7), turned to 90 degrees
- moved Q501 271.0 mm to (117.8, 86.7), turned to 180 degrees
- moved C503 270.7 mm to (116.8, 91.8), turned to 90 degrees
- moved D403 264.8 mm to (120.1, 82.2), turned to 270 degrees
- moved D402 258.8 mm to (126.2, 84.5)
- moved D404 258.5 mm to (121.6, 85.5)
- moved R501 255.8 mm to (114.4, 89.7), turned to 90 degrees
- moved R503 255.0 mm to (114.4, 85.6), turned to 90 degrees
- moved D401 253.9 mm to (126.2, 81.2), turned to 180 degrees
- moved TP301 235.3 mm to (127.5, 61.1)
- moved Q302 233.0 mm to (122.8, 60.1), turned to 270 degrees
- moved C301 225.5 mm to (127.5, 64.9), turned to 90 degrees
- moved R304 220.7 mm to (118.1, 60.1), turned to 90 degrees
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Routing:
- net /Mixer/IF_UNFILT_OUT: track 0.00 -> 19.5 mm
- net Net-(C301-Pad2): track 0.00 -> 14.2 mm
- net Net-(D402-Pad1): track 0.00 -> 12.8 mm, vias 0 -> 2
- net Net-(D401-Pad2): track 0.00 -> 8.67 mm
- net Net-(C503-Pad2): track 0.00 -> 8.43 mm
- net Net-(C502-Pad1): track 0.00 -> 7.11 mm
- net Net-(C303-Pad1): track 0.00 -> 5.85 mm
- net Net-(D401-Pad1): track 0.00 -> 3.31 mm
- net +5V: track 1.52 -> 4.78 mm, vias 1 -> 3
- net /IF Amplifier/IF_AMP_IN: track 0.00 -> 3.06 mm
- net Net-(D403-Pad2): track 0.00 -> 2.49 mm
- net GNDA: track 0.00 -> 2.35 mm, vias 1 -> 2
- net /RF Preamp/PREAMP_OUT: track 0.00 -> 2.29 mm

Commit message: More pcb work
Parts:
- removed J101: CAL_O, footprints:TE_5-1634503-1
- removed J102: CAL_S, footprints:TE_5-1634503-1
- removed J103: CAL_L, footprints:TE_5-1634503-1
- removed R101: 50Ω, Resistor_SMD:R_1206_3216Metric_Pad1.42x1.75mm_HandSolder
- added TP1: TestPoint, TestPoint:TestPoint_Pad_2.5x2.5mm, F.Cu at (68.0, 61.1)
- added TP2: TP_Preamp_Out, TestPoint:TestPoint_Pad_2.5x2.5mm, F.Cu at (106.6, 59.6)
- added TP3: TP_IF_Out, TestPoint:TestPoint_Pad_2.5x2.5mm, F.Cu at (115.8, 88.5)
- added TP4: TP_LO_Pot_Divider, TestPoint:TestPoint_Pad_2.5x2.5mm, F.Cu at (80.5, 78.9)
- added TP5: TP_LO_Out, TestPoint:TestPoint_Pad_2.5x2.5mm, F.Cu at (97.2, 87.0)
- added TP6: TP_LO_Static_Divider, TestPoint:TestPoint_Pad_2.5x2.5mm, F.Cu at (56.6, 69.7)
- added TP7: TP_IF_Amp_In, TestPoint:TestPoint_Pad_2.5x2.5mm, F.Cu at (115.8, 93.4)
- TP501: value TP_Preamp_Out -> TP_IF_Amp_Out
- moved C1 380.7 mm to (57.9, 79.4), turned to 180 degrees
- moved L1 376.0 mm to (57.9, 82.9), turned to 180 degrees
- moved C2 372.9 mm to (61.2, 80.9), turned to 90 degrees
- moved Q1 366.8 mm to (67.3, 94.3)
- moved C402 365.2 mm to (74.6, 90.6), turned to 180 degrees
- moved Q3 364.4 mm to (74.4, 85.7)
- moved C6 361.6 mm to (74.8, 79.5), turned to 270 degrees
- moved Q2 359.1 mm to (67.3, 87.2)
- moved C3 354.6 mm to (60.7, 86.5), turned to 90 degrees
- moved R3 354.1 mm to (63.3, 82.9), turned to 270 degrees
- moved C405 346.4 mm to (75.9, 99.0), turned to 270 degrees
- moved R401 344.7 mm to (53.2, 68.0), turned to 270 degrees
- moved D2 340.3 mm to (53.2, 80.0)
- moved D1 340.3 mm to (53.2, 78.8)
- moved U402 336.7 mm to (86.1, 95.6), turned to 270 degrees
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Routing:
- net -12V: track 0.00 -> 86.9 mm, vias 0 -> 2
- net +12V: track 0.00 -> 75.1 mm, vias 0 -> 1
- net Net-(T401-Pad1): track 0.00 -> 67.0 mm, vias 0 -> 2
- net GND: track 0.00 -> 35.7 mm, vias 0 -> 15
- net Net-(D403-Pad2): track 2.49 -> 36.7 mm
- net Net-(D401-Pad1): track 3.31 -> 36.4 mm
- net Net-(R2-Pad2): track 0.00 -> 29.7 mm
- net Net-(RV401-Pad2): track 0.00 -> 26.8 mm
- net Net-(C1-Pad1): track 0.00 -> 26.5 mm
- net /RF Preamp/PREAMP_OUT: track 2.29 -> 27.4 mm
- net Net-(C5-Pad2): track 0.00 -> 24.6 mm
- net (no net): track 0.00 -> 22.6 mm
- net /Mixer/IF_UNFILT_OUT: track 19.5 -> 37.7 mm
- net Net-(R401-Pad2): track 0.00 -> 15.4 mm
- net Net-(RV401-Pad3): track 0.00 -> 14.8 mm
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- added copper zone on B.Cu, net GND
Other:
- board text added: "THIS STILL NEEDS A POWER BUTTON"
- board text removed: "CAL_LOAD"
- board text removed: "CAL_OPEN"
- board text removed: "CAL_SHORT"

Commit message: First spin of board complete
Parts:
- removed J701: Conn_WallPlug_Earth, TerminalBlock:TerminalBlock_bornier-3_P5.08mm
- added C701: 10uF, Capacitor_THT:CP_Radial_D5.0mm_P2.50mm, F.Cu at (130.0, 107.1)
- added C702: 0.33uF, Capacitor_SMD:C_0805_2012Metric_Pad1.15x1.40mm_HandSolder, F.Cu at (141.2, 128.7)
- added C703: 0.1uF, Capacitor_SMD:C_0805_2012Metric_Pad1.15x1.40mm_HandSolder, F.Cu at (141.2, 121.8)
- added C704: 0.33uF, Capacitor_SMD:C_0805_2012Metric_Pad1.15x1.40mm_HandSolder, F.Cu at (141.2, 116.7)
- added C705: 0.1uF, Capacitor_SMD:C_0805_2012Metric_Pad1.15x1.40mm_HandSolder, F.Cu at (141.2, 133.8)
- added C706: 0.33uF, Capacitor_SMD:C_0805_2012Metric_Pad1.15x1.40mm_HandSolder, F.Cu at (141.2, 140.9)
- added C707: 0.1uF, Capacitor_SMD:C_0805_2012Metric_Pad1.15x1.40mm_HandSolder, F.Cu at (141.2, 145.9)
- added C708: 10uF, Capacitor_THT:CP_Radial_D5.0mm_P2.50mm, F.Cu at (136.9, 104.5)
- added C801: 0.22uF, Capacitor_THT:CP_Radial_D5.0mm_P2.50mm, F.Cu at (96.5, 93.9)
- added C802: 1000uF, Capacitor_THT:CP_Radial_D10.0mm_P5.00mm, F.Cu at (111.0, 90.3)
- added C803: 100uF, Capacitor_THT:CP_Radial_D5.0mm_P2.50mm, F.Cu at (95.5, 82.2)
- added C804: 100uF, Capacitor_THT:CP_Radial_D5.0mm_P2.50mm, F.Cu at (102.3, 93.9)
- added D702: 1N4001, Diode_SMD:D_0805_2012Metric_Pad1.15x1.40mm_HandSolder, F.Cu at (134.3, 131.7)
- added D703: 1N4001, Diode_SMD:D_0805_2012Metric_Pad1.15x1.40mm_HandSolder, F.Cu at (134.3, 140.9)
- added F702: 1.5A Fuse, Fuse:Fuse_0805_2012Metric_Pad1.15x1.40mm_HandSolder, F.Cu at (133.3, 116.5)
- added J801: AudioJack3, Connector_Audio:Jack_3.5mm_Switronic_ST-005-G_horizontal, F.Cu at (57.9, 101.2)
- added LS801: PLS-P830985, Connector_PinSocket_2.54mm:PinSocket_1x02_P2.54mm_Vertical, F.Cu at (120.9, 90.3)
- added P701: Conn_WallPlug_Earth, Sensor_Current:Diodes_SIP-3_4.1x1.5mm_P2.65mm, F.Cu at (57.1, 110.6)
- added R801: 1k, Resistor_THT:R_Axial_DIN0207_L6.3mm_D2.5mm_P10.16mm_Horizontal, F.Cu at (96.5, 90.3)
- added R802: 1k, Resistor_THT:R_Axial_DIN0207_L6.3mm_D2.5mm_P10.16mm_Horizontal, F.Cu at (111.0, 80.9)
- added R803: 1k, Resistor_THT:R_Axial_DIN0207_L6.3mm_D2.5mm_P10.16mm_Horizontal, F.Cu at (111.0, 77.6)
- added SW701: SW_Push_DPDT, Connector_PinSocket_2.54mm:PinSocket_1x06_P2.54mm_Vertical, F.Cu at (126.7, 110.5)
- added U701: L7805CV, Package_TO_SOT_THT:TO-220-3_Vertical, F.Cu at (144.5, 115.7)
- added U702: L7805CV, Package_TO_SOT_THT:TO-220-3_Vertical, F.Cu at (144.5, 127.6)
- added U703: L7805CV, Package_TO_SOT_THT:TO-220-3_Vertical, F.Cu at (144.5, 139.8)
- added U801: LM386, Package_DIP:DIP-8_W7.62mm, F.Cu at (107.2, 85.7)
- added VR701: ECL30UD01-E, footprints:ECL30UD01-E, F.Cu at (89.1, 127.4)
- D701: value GBU606 -> 1N4001; footprint Diode_THT:Diode_Bridge_Vishay_GBU -> Diode_SMD:D_0805_2012Metric_Pad1.15x1.40mm_HandSolder
- F701: value Fuse -> 1.5A Fuse
- TP1: value TestPoint -> Input
- moved C406 95.7 mm to (56.3, 75.1), turned to 180 degrees
- moved D701 82.1 mm to (135.1, 120.5), turned to 270 degrees
- moved C403 79.5 mm to (71.8, 75.5), turned to 270 degrees
- moved F701 57.7 mm to (131.0, 116.5), turned to 270 degrees
- moved C404 55.7 mm to (77.4, 106.8), turned to 180 degrees
- moved NT701 54.2 mm to (118.1, 138.4), turned to 180 degrees
- moved T402 47.9 mm to (140.7, 96.2), turned to 90 degrees
- moved C601 47.6 mm to (130.0, 85.7), turned to 180 degrees
- moved C603 42.4 mm to (133.6, 87.8)
- moved R605 36.5 mm to (126.7, 86.8), turned to 270 degrees
- moved D403 35.4 mm to (145.5, 84.2), turned to 90 degrees
- moved D401 32.0 mm to (140.7, 84.2), turned to 270 degrees
- moved C602 28.4 mm to (130.0, 83.5)
- moved C502 26.7 mm to (102.8, 73.0)
- moved C503 26.7 mm to (115.7, 72.1)
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Connections:
- net /AM Demodulater/DEMOD_OUT renamed /Audio Amp/Audio_In
- net /RF Preamp/RF_IN renamed /InputBandpassFilter/RF_FILTERED_OUT
- D701 pad 1: /Power Supply/DC_REC- -> +12V
- D701 pad 2: /Power Supply/TRANS_AC_P -> +5V
- F701 pad 2: Net-(F701-Pad2) -> /Power Supply/+Power_Pre_Fuse
- NT701 pad 1: Earth -> /Power Supply/Star_Ground
Routing:
- net +12V: track 75.1 -> 234.7 mm, vias 1 -> 4
- net /Audio Amp/Audio_In: track 0.00 -> 117.6 mm, vias 0 -> 1
- net Net-(J801-PadR): track 0.00 -> 100.1 mm
- net +5VP: track 0.00 -> 88.3 mm, vias 0 -> 2
- net -12V: track 86.9 -> 161.1 mm, vias 2 -> 5
- net GND: track 35.7 -> 87.5 mm, vias 15 -> 26
- net /Mixer/IF_UNFILT_OUT: track 37.7 -> 84.8 mm, vias 0 -> 2
- net Net-(P701-Pad1): track 0.00 -> 37.6 mm
- net /Power Supply/+Power_Pre_Fuse: track 0.00 -> 32.2 mm
- net /RF Preamp/PREAMP_OUT: track 27.4 -> 52.7 mm, vias 0 -> 4
- net (no net): track 22.6 -> 0.00 mm
- net Net-(C802-Pad1): track 0.00 -> 20.8 mm
- net Net-(D402-Pad1): track 4.83 -> 23.9 mm, vias 0 -> 2
- net /Power Supply/-Power_Pre_Fuse: track 0.00 -> 18.0 mm, vias 0 -> 1
- net +5VD: track 0.00 -> 12.7 mm
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Other:
- board text added: "AM Radio"
- board text added: "Board Rev: A"
- board text added: "Design & Layout by Skye and Maxwell Ernst"
- board text added: "Schematic Rev: A"
- board text removed: "THIS STILL NEEDS A POWER BUTTON"
