File: AM Radio/BPfilt.sch (KiCad schematic (older format))
At the start: 16 parts

Commit message: Started work on PCB, annotated schematics
Parts:
- gave numbers to parts that had none: 16
Changed lines of the file:
@@
 $EndDescr
 $Comp
-L Device:C_Small C?
+L Device:C_Small C201
 U 1 1 602B441A
 P 3500 3950
-F 0 "C?" V 3271 3950 50  0000 C CNN
+F 0 "C201" V 3271 3950 50  0000 C CNN
 F 1 "4.7nF" V 3362 3950 50  0000 C CNN
 F 2 "Capacitor_SMD:C_0805_2012Metric_Pad1.15x1.40mm_HandSolder" H 3500 3950 50  0001 C CNN
@@
 $EndComp
 $Comp
-L Device:L L?
+L Device:L L203
 U 1 1 602B533C
 P 4000 3950
-F 0 "L?" V 4190 3950 50  0000 C CNN
+F 0 "L203" V 4190 3950 50  0000 C CNN
 F 1 "6.8µH" V 4099 3950 50  0000 C CNN
 F 2 "Inductor_SMD:L_0805_2012Metric_Pad1.15x1.40mm_HandSolder" H 4000 3950 50  0001 C CNN
@@
 	5600 4500 5600 4350
 $Comp
-L Device:C_Small C?
+L Device:C_Small C205
 U 1 1 602B861A
 P 4300 4150
-F 0 "C?" H 4100 4100 50  0000 C CNN
+F 0 "C205" H 4100 4100 50  0000 C CNN
 F 1 "3nF" H 4100 4200 50  0000 C CNN
 F 2 "Capacitor_SMD:C_0805_2012Metric_Pad1.15x1.40mm_HandSolder" H 4300 4150 50  0001 C CNN
@@
 	4300 4250 4300 4350
 $Comp
-L Device:L L?
+L Device:L L207
 U 1 1 602BA889
 P 4700 4150
-F 0 "L?" H 4850 4200 50  0000 C CNN
+F 0 "L207" H 4850 4200 50  0000 C CNN
 F 1 "10µH" H 4850 4100 50  0000 C CNN
 F 2 "Inductor_SMD:L_0805_2012Metric_Pad1.15x1.40mm_HandSolder" H 4700 4150 50  0001 C CNN
@@
 Connection ~ 4300 3950
 $Comp
-L Device:C_Small C?
+L Device:C_Small C202
 U 1 1 602BC43D
 P 5000 3950
-F 0 "C?" V 4771 3950 50  0000 C CNN
+F 0 "C202" V 4771 3950 50  0000 C CNN
 F 1 "2.7nF" V 4862 3950 50  0000 C CNN
 F 2 "Capacitor_SMD:C_0805_2012Metric_Pad1.15x1.40mm_HandSolder" H 5000 3950 50  0001 C CNN
@@
 Connection ~ 4700 3950
 $Comp
-L Device:L L?
+L Device:L L201
 U 1 1 602BCC15
 P 5350 3700
-F 0 "L?" V 5540 3700 50  0000 C CNN
+F 0 "L201" V 5540 3700 50  0000 C CNN
 F 1 "22µH" V 5449 3700 50  0000 C CNN
 F 2 "Inductor_SMD:L_0805_2012Metric_Pad1.15x1.40mm_HandSolder" H 5350 3700 50  0001 C CNN
@@
 	5100 3950 5150 3950
 $Comp
-L Device:C_Small C?
+L Device:C_Small C206
 U 1 1 602BD1F4
 P 5600 4150
-F 0 "C?" H 5400 4100 50  0000 C CNN
+F 0 "C206" H 5400 4100 50  0000 C CNN
 F 1 "3.3nF" H 5400 4200 50  0000 C CNN
 F 2 "Capacitor_SMD:C_0805_2012Metric_Pad1.15x1.40mm_HandSolder" H 5600 4150 50  0001 C CNN
@@
 Connection ~ 4700 4350
 $Comp
-L Device:L L?
+L Device:L L208
 U 1 1 602BE628
 P 5950 4150
-F 0 "L?" H 6100 4200 50  0000 C CNN
+F 0 "L208" H 6100 4200 50  0000 C CNN
 F 1 "10µH" H 6100 4100 50  0000 C CNN
 F 2 "Inductor_SMD:L_0805_2012Metric_Pad1.15x1.40mm_HandSolder" H 5950 4150 50  0001 C CNN
@@
 Connection ~ 5600 4350
 $Comp
-L Device:C_Small C?
+L Device:C_Small C203
 U 1 1 602BF98F
 P 6250 3950
-F 0 "C?" V 6021 3950 50  0000 C CNN
+F 0 "C203" V 6021 3950 50  0000 C CNN
 F 1 "2.7nF" V 6112 3950 50  0000 C CNN
 F 2 "Capacitor_SMD:C_0805_2012Metric_Pad1.15x1.40mm_HandSolder" H 6250 3950 50  0001 C CNN
@@
 	6350 3950 6400 3950
 $Comp
-L Device:C_Small C?
+L Device:C_Small C207
 U 1 1 602C060F
 P 6850 4150
-F 0 "C?" H 6650 4100 50  0000 C CNN
+F 0 "C207" H 6650 4100 50  0000 C CNN
 F 1 "3nF" H 6650 4200 50  0000 C CNN
 F 2 "Capacitor_SMD:C_0805_2012Metric_Pad1.15x1.40mm_HandSolder" H 6850 4150 50  0001 C CNN
@@
 $EndComp
 $Comp
-L Device:L L?
+L Device:L L209
 U 1 1 602C0615
 P 7250 4150
-F 0 "L?" H 7400 4200 50  0000 C CNN
+F 0 "L209" H 7400 4200 50  0000 C CNN
 F 1 "10µH" H 7400 4100 50  0000 C CNN
 F 2 "Inductor_SMD:L_0805_2012Metric_Pad1.15x1.40mm_HandSolder" H 7250 4150 50  0001 C CNN
@@
 Connection ~ 6850 3950
 $Comp
-L Device:C_Small C?
+L Device:C_Small C204
 U 1 1 602C4200
 P 7500 3950
-F 0 "C?" V 7271 3950 50  0000 C CNN
+F 0 "C204" V 7271 3950 50  0000 C CNN
 F 1 "4.7nF" V 7362 3950 50  0000 C CNN
 F 2 "Capacitor_SMD:C_0805_2012Metric_Pad1.15x1.40mm_HandSolder" H 7500 3950 50  0001 C CNN
@@
 $EndComp
 $Comp
-L Device:L L?
+L Device:L L206
 U 1 1 602C4206
 P 8000 3950
-F 0 "L?" V 8190 3950 50  0000 C CNN
+F 0 "L206" V 8190 3950 50  0000 C CNN
 F 1 "6.8µH" V 8099 3950 50  0000 C CNN
 F 2 "Inductor_SMD:L_0805_2012Metric_Pad1.15x1.40mm_HandSolder" H 8000 3950 50  0001 C CNN
@@
 	8150 3950 8700 3950
 $Comp
-L Device:L L?
+L Device:L L204
 U 1 1 602C6235
 P 5350 3950
-F 0 "L?" V 5540 3950 50  0000 C CNN
+F 0 "L204" V 5540 3950 50  0000 C CNN
 F 1 "22µH" V 5449 3950 50  0000 C CNN
 F 2 "Inductor_SMD:L_0805_2012Metric_Pad1.15x1.40mm_HandSolder" H 5350 3950 50  0001 C CNN
@@
 	5600 3700 5500 3700
 $Comp
-L Device:L L?
+L Device:L L202
 U 1 1 602C8F35
 P 6600 3700
-F 0 "L?" V 6790 3700 50  0000 C CNN
+F 0 "L202" V 6790 3700 50  0000 C CNN
 F 1 "22µH" V 6699 3700 50  0000 C CNN
 F 2 "Inductor_SMD:L_0805_2012Metric_Pad1.15x1.40mm_HandSolder" H 6600 3700 50  0001 C CNN
@@
 $EndComp
 $Comp
-L Device:L L?
+L Device:L L205
 U 1 1 602C8F3B
 P 6600 3950
-F 0 "L?" V 6790 3950 50  0000 C CNN
+F 0 "L205" V 6790 3950 50  0000 C CNN
 F 1 "22µH" V 6699 3950 50  0000 C CNN
 F 2 "Inductor_SMD:L_0805_2012Metric_Pad1.15x1.40mm_HandSolder" H 6600 3950 50  0001 C CNN
@@
 RF_OUT_FILTERED
 $Comp
-L power:GNDA #PWR?
+L power:GNDA #PWR0108
 U 1 1 6058FCC7
 P 5600 4500
-F 0 "#PWR?" H 5600 4250 50  0001 C CNN
+F 0 "#PWR0108" H 5600 4250 50  0001 C CNN
 F 1 "GNDA" H 5605 4327 50  0000 C CNN
 F 2 "" H 5600 4500 50  0001 C CNN

Commit message: First spin of board complete
Connections:
- net RF_OUT_FILTERED renamed RF_FILTERED_OUT
Changed lines of the file:
@@
 $Descr A4 11693 8268
 encoding utf-8
-Sheet 2 7
+Sheet 2 8
 Title ""
-Date ""
-Rev ""
+Date "2021-06-24"
+Rev "A"
 Comp ""
 Comment1 ""
@@
 RF_IN
 Text HLabel 8700 3950 2    50   Output ~ 0
-RF_OUT_FILTERED
+RF_FILTERED_OUT
 $Comp
 L power:GNDA #PWR0108
