File: AM Radio/Demod.sch (KiCad schematic (older format))
At the start: 9 parts

Commit message: Started work on PCB, annotated schematics
Parts:
- C601, C602, C603: renamed from C?; footprint (none) -> Capacitor_SMD:C_0805_2012Metric_Pad1.15x1.40mm_HandSolder
- D601: renamed from D?; footprint (none) -> Diode_SMD:D_0805_2012Metric_Pad1.15x1.40mm_HandSolder
- R601, R602, R603, R604, R605: renamed from R?; footprint (none) -> Resistor_SMD:R_0805_2012Metric_Pad1.15x1.40mm_HandSolder
Changed lines of the file:
@@
 DEMOD_OUT
 $Comp
-L Device:D D?
+L Device:D D601
 U 1 1 606EA642
 P 4600 3000
-F 0 "D?" H 4600 2784 50  0000 C CNN
+F 0 "D601" H 4600 2784 50  0000 C CNN
 F 1 "D" H 4600 2875 50  0000 C CNN
-F 2 "" H 4600 3000 50  0001 C CNN
+F 2 "Diode_SMD:D_0805_2012Metric_Pad1.15x1.40mm_HandSolder" H 4600 3000 50  0001 C CNN
 F 3 "~" H 4600 3000 50  0001 C CNN
 	1    4600 3000
@@
 $EndComp
 $Comp
-L Device:C_Small C?
+L Device:C_Small C602
 U 1 1 606EB908
 P 5000 3200
-F 0 "C?" H 5092 3246 50  0000 L CNN
+F 0 "C602" H 5092 3246 50  0000 L CNN
 F 1 "2.2nF" H 5092 3155 50  0000 L CNN
-F 2 "" H 5000 3200 50  0001 C CNN
+F 2 "Capacitor_SMD:C_0805_2012Metric_Pad1.15x1.40mm_HandSolder" H 5000 3200 50  0001 C CNN
 F 3 "~" H 5000 3200 50  0001 C CNN
 	1    5000 3200
@@
 $EndComp
 $Comp
-L Device:R_Small R?
+L Device:R_Small R604
 U 1 1 606EC38C
 P 5400 3200
-F 0 "R?" H 5459 3246 50  0000 L CNN
+F 0 "R604" H 5459 3246 50  0000 L CNN
 F 1 "10k" V 5400 3150 39  0000 L CNN
-F 2 "" H 5400 3200 50  0001 C CNN
+F 2 "Resistor_SMD:R_0805_2012Metric_Pad1.15x1.40mm_HandSolder" H 5400 3200 50  0001 C CNN
 F 3 "~" H 5400 3200 50  0001 C CNN
 	1    5400 3200
@@
 $EndComp
 $Comp
-L Device:R_Small R?
+L Device:R_Small R602
 U 1 1 606ED541
 P 5750 3000
-F 0 "R?" V 5850 3000 50  0000 C CNN
+F 0 "R602" V 5850 3000 50  0000 C CNN
 F 1 "100k" V 5750 3000 39  0000 C CNN
-F 2 "" H 5750 3000 50  0001 C CNN
+F 2 "Resistor_SMD:R_0805_2012Metric_Pad1.15x1.40mm_HandSolder" H 5750 3000 50  0001 C CNN
 F 3 "~" H 5750 3000 50  0001 C CNN
 	1    5750 3000
@@
 $EndComp
 $Comp
-L Device:C_Small C?
+L Device:C_Small C603
 U 1 1 606ED905
 P 6000 3200
-F 0 "C?" H 6092 3246 50  0000 L CNN
+F 0 "C603" H 6092 3246 50  0000 L CNN
 F 1 "1nF" H 6092 3155 50  0000 L CNN
-F 2 "" H 6000 3200 50  0001 C CNN
+F 2 "Capacitor_SMD:C_0805_2012Metric_Pad1.15x1.40mm_HandSolder" H 6000 3200 50  0001 C CNN
 F 3 "~" H 6000 3200 50  0001 C CNN
 	1    6000 3200
@@
 $EndComp
 $Comp
-L Device:C_Small C?
+L Device:C_Small C601
 U 1 1 606EDE43
 P 6300 3000
-F 0 "C?" V 6529 3000 50  0000 C CNN
+F 0 "C601" V 6529 3000 50  0000 C CNN
 F 1 "1nF" V 6438 3000 50  0000 C CNN
-F 2 "" H 6300 3000 50  0001 C CNN
+F 2 "Capacitor_SMD:C_0805_2012Metric_Pad1.15x1.40mm_HandSolder" H 6300 3000 50  0001 C CNN
 F 3 "~" H 6300 3000 50  0001 C CNN
 	1    6300 3000
@@
 $EndComp
 $Comp
-L Device:R_Small R?
+L Device:R_Small R605
 U 1 1 606EE068
 P 6700 3200
-F 0 "R?" H 6759 3246 50  0000 L CNN
+F 0 "R605" H 6759 3246 50  0000 L CNN
 F 1 "1M" H 6759 3155 50  0000 L CNN
-F 2 "" H 6700 3200 50  0001 C CNN
+F 2 "Resistor_SMD:R_0805_2012Metric_Pad1.15x1.40mm_HandSolder" H 6700 3200 50  0001 C CNN
 F 3 "~" H 6700 3200 50  0001 C CNN
 	1    6700 3200
@@
 $EndComp
 $Comp
-L power:GND #PWR?
+L power:GND #PWR0134
 U 1 1 606EE4ED
 P 5200 3400
-F 0 "#PWR?" H 5200 3150 50  0001 C CNN
+F 0 "#PWR0134" H 5200 3150 50  0001 C CNN
 F 1 "GND" H 5205 3227 50  0000 C CNN
 F 2 "" H 5200 3400 50  0001 C CNN
@@
 	6000 3000 6000 3100
 $Comp
-L power:GND #PWR?
+L power:GND #PWR0135
 U 1 1 606EFBA8
 P 6000 3350
-F 0 "#PWR?" H 6000 3100 50  0001 C CNN
+F 0 "#PWR0135" H 6000 3100 50  0001 C CNN
 F 1 "GND" H 6005 3177 50  0000 C CNN
 F 2 "" H 6000 3350 50  0001 C CNN
@@
 	6700 3000 6700 3100
 $Comp
-L power:GND #PWR?
+L power:GND #PWR0136
 U 1 1 606F04D4
 P 6700 3350
-F 0 "#PWR?" H 6700 3100 50  0001 C CNN
+F 0 "#PWR0136" H 6700 3100 50  0001 C CNN
 F 1 "GND" H 6705 3177 50  0000 C CNN
 F 2 "" H 6700 3350 50  0001 C CNN
@@
 Connection ~ 6000 3000
 $Comp
-L Device:R_Small R?
+L Device:R_Small R601
 U 1 1 606F11C8
 P 4200 2850
-F 0 "R?" V 4300 2850 50  0000 C CNN
+F 0 "R601" V 4300 2850 50  0000 C CNN
 F 1 "100k" V 4200 2850 39  0000 C CNN
-F 2 "" H 4200 2850 50  0001 C CNN
+F 2 "Resistor_SMD:R_0805_2012Metric_Pad1.15x1.40mm_HandSolder" H 4200 2850 50  0001 C CNN
 F 3 "~" H 4200 2850 50  0001 C CNN
 	1    4200 2850
@@
 	3950 3000 4200 3000
 $Comp
-L Device:R_Small R?
+L Device:R_Small R603
 U 1 1 606F25F6
 P 4200 3150
-F 0 "R?" V 4300 3150 50  0000 C CNN
+F 0 "R603" V 4300 3150 50  0000 C CNN
 F 1 "33k" V 4200 3150 39  0000 C CNN
-F 2 "" H 4200 3150 50  0001 C CNN
+F 2 "Resistor_SMD:R_0805_2012Metric_Pad1.15x1.40mm_HandSolder" H 4200 3150 50  0001 C CNN
 F 3 "~" H 4200 3150 50  0001 C CNN
 	1    4200 3150
@@
 	4200 3000 4200 2950
 $Comp
-L power:+5V #PWR?
+L power:+5V #PWR0137
 U 1 1 606F2E7F
 P 4200 2700
-F 0 "#PWR?" H 4200 2550 50  0001 C CNN
+F 0 "#PWR0137" H 4200 2550 50  0001 C CNN
 F 1 "+5V" H 4215 2873 50  0000 C CNN
 F 2 "" H 4200 2700 50  0001 C CNN
@@
 	4200 3300 4200 3250
 $Comp
-L power:GND #PWR?
+L power:GND #PWR0138
 U 1 1 606F3582
 P 4200 3300
-F 0 "#PWR?" H 4200 3050 50  0001 C CNN
+F 0 "#PWR0138" H 4200 3050 50  0001 C CNN
 F 1 "GND" H 4205 3127 50  0000 C CNN
 F 2 "" H 4200 3300 50  0001 C CNN
