File: AM Radio/Mixer.sch (KiCad schematic (older format))
At the start: 36 parts, among them Q1 2N2222, Q2 2N2222, Q3 2N2222, U1 OPAMP

Commit message: Added part numbers for mixer OPAMPs
Parts:
- U1, U? (x2): value OPAMP -> AD711
Changed lines of the file:
@@
 P 6600 2300
 F 0 "U1" H 6944 2346 50  0000 L CNN
-F 1 "OPAMP" H 6944 2255 50  0000 L CNN
+F 1 "AD711" H 6944 2255 50  0000 L CNN
 F 2 "" H 6600 2300 50  0001 C CNN
 F 3 "~" H 6600 2300 50  0001 C CNN
@@
 P 1450 4050
 F 0 "U?" H 1700 4250 50  0000 L CNN
-F 1 "OPAMP" H 1700 4150 50  0000 L CNN
+F 1 "AD711" H 1700 4150 50  0000 L CNN
 F 2 "" H 1450 4050 50  0001 C CNN
 F 3 "~" H 1450 4050 50  0001 C CNN
@@
 P 2950 3900
 F 0 "U?" H 3200 4100 50  0000 L CNN
-F 1 "OPAMP" H 3200 4000 50  0000 L CNN
+F 1 "AD711" H 3200 4000 50  0000 L CNN
 F 2 "" H 2950 3900 50  0001 C CNN
 F 3 "~" H 2950 3900 50  0001 C CNN

Commit message: Added new buffer parts for mixer
Parts:
- removed U1, U? (x2): AD711, symbol pspice:OPAMP
- added C?: 0.1uF, symbol Device:C_Small
- added U? (x3): AD711, Package_DIP:DIP-8_W7.62mm_LongPads, symbol CustomComponents:AD711
Connections:
- wire segments 130 -> 129
Other:
- note added: "AM Radio Local Oscillator 960Khz to 2.1Mhz"
- note removed: "AM Radio Local Oscillator ~960Khz to 2.1Mhz"
- note removed: "which opamp?"
- moved on the sheet: C1, C2, C3, C4, C5, C6, C?, D1, D2, D?, L1, Q1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

Commit message: Started work on PCB, annotated schematics
Parts:
- C1, C2, C3, C4, C5, C6: footprint (none) -> Capacitor_SMD:C_0805_2012Metric_Pad1.15x1.40mm_HandSolder
- C401, C402, C403, C404, C405, C406: renamed from C?; footprint (none) -> Capacitor_SMD:C_0805_2012Metric_Pad1.15x1.40mm_HandSolder
- D1, D2: footprint (none) -> Capacitor_SMD:C_0402_1005Metric
- D401, D402, D403, D404: renamed from D?; footprint (none) -> Diode_SMD:D_0805_2012Metric_Pad1.15x1.40mm_HandSolder
- L1: footprint (none) -> Inductor_SMD:L_0805_2012Metric_Pad1.15x1.40mm_HandSolder
- Q1, Q2, Q3: footprint (none) -> Package_TO_SOT_SMD:SOT-23
- R1, R2, R3, R4, R5, R6, R7: footprint (none) -> Resistor_SMD:R_0805_2012Metric_Pad1.15x1.40mm_HandSolder
- R401, R402: renamed from R?; footprint (none) -> Resistor_SMD:R_0805_2012Metric_Pad1.15x1.40mm_HandSolder
- RV401: renamed from RV?; footprint (none) -> Potentiometer_THT:Potentiometer_Bourns_3266W_Vertical
- gave numbers to parts that had none: 5

Commit message: More pcb work
Parts:
- added TP3: TP_IF_Out, TestPoint:TestPoint_Pad_2.5x2.5mm, symbol Connector:TestPoint
- added TP4: TP_LO_Pot_Divider, TestPoint:TestPoint_Pad_2.5x2.5mm, symbol Connector:TestPoint
- added TP5: TP_LO_Out, TestPoint:TestPoint_Pad_2.5x2.5mm, symbol Connector:TestPoint
- added TP6: TP_LO_Static_Divider, TestPoint:TestPoint_Pad_2.5x2.5mm, symbol Connector:TestPoint
Connections:
- net IF_UNFILT_OUT: now also TP3.1
- net at T401.1 (P1), U401.6: now also TP5.1
- net at RV401.2, U402.3 (+): now also TP4.1
- net at R401.2, R402.1, U403.3 (+): now also TP6.1
Changed lines of the file:
@@
 	12300 4100 12200 4100
 Wire Wire Line
-	12200 4100 12200 4450
+	12200 4100 12200 4300
 Wire Wire Line
 	12200 4450 12250 4450
@@
 U 1 1 60849931
 P 4600 5450
-F 0 "C404" H 4400 5500 50  0000 L CNN
+F 0 "C404" H 4300 5500 50  0000 L CNN
 F 1 "0.1uF" H 4300 5400 50  0000 L CNN
 F 2 "Capacitor_SMD:C_0805_2012Metric_Pad1.15x1.40mm_HandSolder" H 4600 5450 50  0001 C CNN
@@
 	8300 4450 8300 4500
 Wire Wire Line
-	9000 4000 9550 4000
+	9000 4000 9350 4000
 $Comp
 L CustomComponents:AD711 U401
@@
 Connection ~ 5400 5900
 Wire Wire Line
-	3700 5800 4100 5800
+	3700 5800 3950 5800
 Wire Wire Line
 	2900 6050 2950 6050
@@
 Wire Wire Line
 	2200 5000 2200 5650
+$Comp
+L Connector:TestPoint TP?
+U 1 1 60C0401A
+P 11950 4850
+AR Path="/6053DD24/60C0401A" Ref="TP?"  Part="1"
+AR Path="/60594038/60C0401A" Ref="TP3"  Part="1"
+F 0 "TP3" V 12150 4850 50  0000 L CNN
+F 1 "TP_IF_Out" V 12050 4850 50  0000 L CNN
+F 2 "TestPoint:TestPoint_Pad_2.5x2.5mm" H 12150 4850 50  0001 C CNN
+F 3 "~" H 12150 4850 50  0001 C CNN
+	1    11950 4850
+	0    -1   -1   0
+$EndComp
+Wire Wire Line
+	11950 4850 12100 4850
+Wire Wire Line
+	12100 4850 12100 4300
+Wire Wire Line
+	12100 4300 12200 4300
+Connection ~ 12200 4300
+Wire Wire Line
+	12200 4300 12200 4450
+$Comp
+L Connector:TestPoint TP?
+U 1 1 60C104E8
+P 1300 5950
+AR Path="/6053DD24/60C104E8" Ref="TP?"  Part="1"
+AR Path="/60594038/60C104E8" Ref="TP6"  Part="1"
+F 0 "TP6" V 1500 5950 50  0000 L CNN
+F 1 "TP_LO_Static_Divider" V 1400 5950 50  0000 L CNN
+F 2 "TestPoint:TestPoint_Pad_2.5x2.5mm" H 1500 5950 50  0001 C CNN
+F 3 "~" H 1500 5950 50  0001 C CNN
+	1    1300 5950
+	0    -1   -1   0
+$EndComp
+Wire Wire Line
+	1300 5950 1400 5950
+$Comp
+L Connector:TestPoint TP?
+U 1 1 60C21E7F
+P 3900 5200
+AR Path="/6053DD24/60C21E7F" Ref="TP?"  Part="1"
+AR Path="/60594038/60C21E7F" Ref="TP4"  Part="1"
+F 0 "TP4" V 4100 5200 50  0000 L CNN
+F 1 "TP_LO_Pot_Divider" V 4000 5200 50  0000 L CNN
+F 2 "TestPoint:TestPoint_Pad_2.5x2.5mm" H 4100 5200 50  0001 C CNN
+F 3 "~" H 4100 5200 50  0001 C CNN
+	1    3900 5200
+	0    -1   -1   0
+$EndComp
+Wire Wire Line
+	3900 5200 3950 5200
+Wire Wire Line
+	3950 5200 3950 5800
+Connection ~ 3950 5800
+Wire Wire Line
+	3950 5800 4100 5800
+$Comp
+L Connector:TestPoint TP?
+U 1 1 60C2E679
+P 9300 5200
+AR Path="/6053DD24/60C2E679" Ref="TP?"  Part="1"
+AR Path="/60594038/60C2E679" Ref="TP5"  Part="1"
+F 0 "TP5" V 9500 5200 50  0000 L CNN
+F 1 "TP_LO_Out" V 9400 5200 50  0000 L CNN
+F 2 "TestPoint:TestPoint_Pad_2.5x2.5mm" H 9500 5200 50  0001 C CNN
+F 3 "~" H 9500 5200 50  0001 C CNN
+	1    9300 5200
+	0    -1   -1   0
+$EndComp
+Wire Wire Line
+	9300 5200 9350 5200
+Wire Wire Line
+	9350 5200 9350 4000
+Connection ~ 9350 4000
+Wire Wire Line
+	9350 4000 9550 4000
 $EndSCHEMATC
