File: AM Radio/PSU.sch (KiCad schematic (older format))
At the start: 6 parts

Commit message: Started work on PCB, annotated schematics
Parts:
- removed HS? (x2): Heatsink, footprints:VM1-038-1AE, symbol Mechanical:Heatsink_Pad
- F701: renamed from F?; footprint (none) -> Fuse:Fuse_0805_2012Metric_Pad1.15x1.40mm_HandSolder
- J701: renamed from J?; footprint (none) -> TerminalBlock:TerminalBlock_bornier-3_P5.08mm
- NT701: renamed from NT?; footprint (none) -> NetTie:NetTie-3_SMD_Pad2.0mm
- gave numbers to parts that had none: 1
Connections:
- wire segments 17 -> 15
Changed lines of the file:
@@
 $EndDescr
 $Comp
-L Connector:Conn_WallPlug_Earth J?
+L Connector:Conn_WallPlug_Earth J701
 U 1 1 6070A6CF
 P 700 1850
-F 0 "J?" H 767 2084 50  0000 C CNN
+F 0 "J701" H 767 2084 50  0000 C CNN
 F 1 "Conn_WallPlug_Earth" H 767 2084 50  0001 C CNN
-F 2 "" H 1100 1850 50  0001 C CNN
+F 2 "TerminalBlock:TerminalBlock_bornier-3_P5.08mm" H 1100 1850 50  0001 C CNN
 F 3 "~" H 1100 1850 50  0001 C CNN
 	1    700  1850
@@
 $EndComp
 $Comp
-L power:Earth #PWR?
+L power:Earth #PWR0139
 U 1 1 6070C00A
 P 1050 2200
-F 0 "#PWR?" H 1050 1950 50  0001 C CNN
+F 0 "#PWR0139" H 1050 1950 50  0001 C CNN
 F 1 "Earth" H 1050 2050 50  0001 C CNN
 F 2 "" H 1050 2200 50  0001 C CNN
@@
 P 1300 2600
 AR Path="/6070EB69" Ref="#PWR?"  Part="1"
-AR Path="/607045AB/6070EB69" Ref="#PWR?"  Part="1"
-F 0 "#PWR?" H 1300 2350 50  0001 C CNN
+AR Path="/607045AB/6070EB69" Ref="#PWR0140"  Part="1"
+F 0 "#PWR0140" H 1300 2350 50  0001 C CNN
 F 1 "GNDA" H 1305 2427 50  0000 C CNN
 F 2 "" H 1300 2600 50  0001 C CNN
@@
 P 1600 2600
 AR Path="/6070EB71" Ref="#PWR?"  Part="1"
-AR Path="/607045AB/6070EB71" Ref="#PWR?"  Part="1"
-F 0 "#PWR?" H 1600 2350 50  0001 C CNN
+AR Path="/607045AB/6070EB71" Ref="#PWR0141"  Part="1"
+F 0 "#PWR0141" H 1600 2350 50  0001 C CNN
 F 1 "GND" H 1605 2427 50  0000 C CNN
 F 2 "" H 1600 2600 50  0001 C CNN
@@
 $EndComp
 $Comp
-L Device:Net-Tie_3 NT?
+L Device:Net-Tie_3 NT701
 U 1 1 6070EDCF
 P 1450 2450
-F 0 "NT?" H 1450 2631 50  0000 C CNN
+F 0 "NT701" H 1450 2631 50  0000 C CNN
 F 1 "Net-Tie_3" H 1450 2540 50  0000 C CNN
-F 2 "" H 1450 2450 50  0001 C CNN
+F 2 "NetTie:NetTie-3_SMD_Pad2.0mm" H 1450 2450 50  0001 C CNN
 F 3 "~" H 1450 2450 50  0001 C CNN
 	1    1450 2450
@@
 	1000 1750 1050 1750
 $Comp
-L Device:Fuse F?
+L Device:Fuse F701
 U 1 1 5EB5803D
 P 1200 1750
-F 0 "F?" V 1003 1750 50  0000 C CNN
+F 0 "F701" V 1003 1750 50  0000 C CNN
 F 1 "Fuse" V 1094 1750 50  0000 C CNN
-F 2 "" V 1130 1750 50  0001 C CNN
+F 2 "Fuse:Fuse_0805_2012Metric_Pad1.15x1.40mm_HandSolder" V 1130 1750 50  0001 C CNN
 F 3 "~" H 1200 1750 50  0001 C CNN
 	1    1200 1750
@@
 Wire Wire Line
 	1000 1950 1350 1950
-$Comp
-L Mechanical:Heatsink_Pad HS?
-U 1 1 5F8B5226
-P 5800 7400
-F 0 "HS?" H 5942 7521 50  0000 L CNN
-F 1 "Heatsink" H 5942 7430 50  0000 L CNN
-F 2 "footprints:VM1-038-1AE" H 5812 7400 50  0001 C CNN
-F 3 "~" H 5812 7400 50  0001 C CNN
-	1    5800 7400
-	1    0    0    -1
-$EndComp
-$Comp
-L Mechanical:Heatsink_Pad HS?
-U 1 1 5F8B522C
-P 6450 7400
-F 0 "HS?" H 6592 7521 50  0000 L CNN
-F 1 "Heatsink" H 6592 7430 50  0000 L CNN
-F 2 "footprints:VM1-038-1AE" H 6462 7400 50  0001 C CNN
-F 3 "~" H 6462 7400 50  0001 C CNN
-	1    6450 7400
-	1    0    0    -1
-$EndComp
-$Comp
-L power:GND #PWR?
-U 1 1 5F8B5232
-P 5800 7550
-F 0 "#PWR?" H 5800 7300 50  0001 C CNN
-F 1 "GND" H 5805 7377 50  0000 C CNN
-F 2 "" H 5800 7550 50  0001 C CNN
-F 3 "" H 5800 7550 50  0001 C CNN
-	1    5800 7550
-	1    0    0    -1
-$EndComp
-Wire Wire Line
-	5800 7550 5800 7500
-$Comp
-L power:GND #PWR?
-U 1 1 5F8B5239
-P 6450 7550
-F 0 "#PWR?" H 6450 7300 50  0001 C CNN
-F 1 "GND" H 6455 7377 50  0000 C CNN
-F 2 "" H 6450 7550 50  0001 C CNN
-F 3 "" H 6450 7550 50  0001 C CNN
-	1    6450 7550
-	1    0    0    -1
-$EndComp
-Wire Wire Line
-	6450 7550 6450 7500
 Text Label 2500 1950 0    39   ~ 0
 TRANS_AC_N
@@
 TRANS_AC_P
 $Comp
-L Device:D_Bridge_-AA+ D?
+L Device:D_Bridge_-AA+ D701
 U 1 1 5EB58031
 P 2000 1000
-F 0 "D?" H 2200 900 50  0000 L CNN
+F 0 "D701" H 2200 900 50  0000 L CNN
 F 1 "GBU606" H 2200 800 50  0000 L CNN
 F 2 "Diode_THT:Diode_Bridge_Vishay_GBU" H 2000 1000 50  0001 C CNN

Commit message: First spin of board complete
Parts:
- removed D701: GBU606, Diode_THT:Diode_Bridge_Vishay_GBU, symbol Device:D_Bridge_-AA+
- removed J701: Conn_WallPlug_Earth, TerminalBlock:TerminalBlock_bornier-3_P5.08mm, symbol Connector:Conn_WallPlug_Earth
- added C701, C708: 10uF, Capacitor_THT:CP_Radial_D5.0mm_P2.50mm, symbol Device:CP_Small
- added C702, C704, C706: 0.33uF, Capacitor_SMD:C_0805_2012Metric_Pad1.15x1.40mm_HandSolder, symbol Device:C_Small
- added C703, C705, C707: 0.1uF, Capacitor_SMD:C_0805_2012Metric_Pad1.15x1.40mm_HandSolder, symbol Device:C_Small
- added D701, D702, D703: 1N4001, Diode_SMD:D_0805_2012Metric_Pad1.15x1.40mm_HandSolder, symbol Device:D
- added F702: 1.5A Fuse, Fuse:Fuse_0805_2012Metric_Pad1.15x1.40mm_HandSolder, symbol Device:Fuse
- added P701: Conn_WallPlug_Earth, Sensor_Current:Diodes_SIP-3_4.1x1.5mm_P2.65mm, symbol Connector:Conn_WallPlug_Earth
- added SW701: SW_Push_DPDT, Connector_PinSocket_2.54mm:PinSocket_1x06_P2.54mm_Vertical, symbol Switch:SW_Push_DPDT
- added U701, U702, U703: L7805CV, Package_TO_SOT_THT:TO-220-3_Vertical, symbol dk_PMIC-Voltage-Regulators-Linear:L7805CV
- added VR701: ECL30UD01-E, footprints:ECL30UD01-E, symbol CustomComponents:ECL30UD01-E
- F701: value Fuse -> 1.5A Fuse
Connections:
- net labels added: +12V, +5V, +5VD, +5VP, +Power_Pre_Fuse, -12V, -Power_Pre_Fuse, Star_Ground
- net labels removed: DC_REC+, DC_REC-, TRANS_AC_N, TRANS_AC_P
- wire segments 15 -> 90
- no-connect marks 0 -> 2
Other:
- note added: "+5V Rail (Audio Only)"
- note added: "+5V Rail (RF only)"
- note added: "LD30-23B15R2 For positive rails + ? for negative\nOR\nECL30UD01-E For positive + negative with linear front end for RF sections"
- note added: "Power Input"
- note added: "Rail Descriptions:\n\n+12V @ 1.5A \n+5V 100mA (NAME: +5V) (RF ONLY) (700mW)\n+5V @ 100mA (NAME: +5VP) (AUDIO ONLY) (700mW)\n+5V @ 350mA (NAME: +5VD) (DIGITAL + DISPLAY ONLY) (2.45W)\nGND\nGNDA\n-12 @ 100mA"
- note removed: "STAR GROUND"
- moved on the sheet: F701, NT701
